File: megacommand18.brd (EAGLE design)
At the start: 109.8 x 83 mm, 74 parts, among them IC1 74HC573N, IC2 74LS165N, IC3 74LS165N, SW1 PEC11, SW2 PEC11, SW3 PEC11, SW4 PEC11

Commit message: preserve
Parts:
- removed U$11, U$12, U$13, U$2, U$3, U$4, U$5, U$6: ALPHA-ROT-ENCODER, SteMarie:TW-700198
- LED0, LED1: value (none) -> 5mm LED
- moved R13 52.5 mm to (83.5, 60.8), flipped to the bottom
- moved C11 32.6 mm to (98.0, 35.0)
- moved C14 19.7 mm to (98.0, 22.5)
- moved R9 13.5 mm to (75.0, 60.8), turned to 270 degrees
- moved R10 11.4 mm to (77.8, 60.8), turned to 270 degrees
- moved C9 11.2 mm to (77.7, 7.07)
- moved D2 6.50 mm to (54.0, 65.2)
- moved R11 6.25 mm to (65.0, 53.8)
- moved R6 6.25 mm to (72.3, 60.8)
- moved OK2 6.01 mm to (65.0, 61.0)
- moved C13 5.55 mm to (98.0, 3.50)
- moved R3 4.53 mm to (54.8, 19.2), turned to 0 degrees
- moved C3 2.26 mm to (54.8, 7.00)
- moved R2 2.15 mm to (102.2, 24.0)
- moved C2 2.14 mm to (77.8, 18.5)
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Connections:
- removed net N$24: U$2.P3, U$3.P3
- removed net N$25: U$2.P2, U$3.P2
- removed net N$28: U$2.P1, U$3.P1
- removed net N$29: U$2.P5, U$3.P5
- removed net N$30: U$2.P4, U$3.P4
- removed net N$31: U$4.P3, U$5.P3
- removed net N$32: U$4.P2, U$5.P2
- removed net N$33: U$4.P1, U$5.P1
- removed net N$34: U$4.P5, U$5.P5
- removed net N$35: U$4.P4, U$5.P4
- removed net N$36: U$11.P3, U$6.P3
- removed net N$37: U$11.P2, U$6.P2
- removed net N$38: U$11.P1, U$6.P1
- removed net N$39: U$11.P5, U$6.P5
- removed net N$40: U$11.P4, U$6.P4
- removed net N$41: U$12.P3, U$13.P3
- removed net N$42: U$12.P2, U$13.P2
- removed net N$43: U$12.P1, U$13.P1
- removed net N$44: U$12.P5, U$13.P5
- removed net N$45: U$12.P4, U$13.P4
- net PB0: now also JP1.7; no longer U1.2
- net PL6: now also U1.2; no longer JP1.7
Routing:
- net +5V: track 0.00 -> 202.0 mm
- net GND: track 0.00 -> 170.2 mm
- net N$23: track 0.00 -> 83.3 mm
- net VIN: track 0.00 -> 12.1 mm
