File: megacommand18.sch (EAGLE design)
At the start: 73 parts, among them IC1 74HC573N, IC2 74LS165N, IC3 74LS165N, J1 POWER_JACKSLT, SW1 PEC11, SW2 PEC11, SW3 PEC11, SW4 PEC11, U1 AS6C1008-55PCN

Commit message: preserve
Parts:
- removed U$11, U$12, U$13, U$2, U$3, U$4, U$5, U$6: ALPHA-ROT-ENCODER, SteMarie:ALPHA-ROT-ENCODER
- LED0, LED1: value (none) -> 5mm LED
Connections:
- removed net N$24: U$2.A, U$3.A
- removed net N$25: U$2.COM, U$3.COM
- removed net N$28: U$2.B, U$3.B
- removed net N$29: U$2.S2, U$3.S2
- removed net N$30: U$2.S1, U$3.S1
- removed net N$31: U$4.A, U$5.A
- removed net N$32: U$4.COM, U$5.COM
- removed net N$33: U$4.B, U$5.B
- removed net N$34: U$4.S2, U$5.S2
- removed net N$35: U$4.S1, U$5.S1
- removed net N$36: U$11.A, U$6.A
- removed net N$37: U$11.COM, U$6.COM
- removed net N$38: U$11.B, U$6.B
- removed net N$39: U$11.S2, U$6.S2
- removed net N$40: U$11.S1, U$6.S1
- removed net N$41: U$12.A, U$13.A
- removed net N$42: U$12.COM, U$13.COM
- removed net N$43: U$12.B, U$13.B
- removed net N$44: U$12.S2, U$13.S2
- removed net N$45: U$12.S1, U$13.S1
- net PB0: now also JP1.7; no longer U1.A16
- net PL6: now also U1.A16; no longer JP1.7
